File: pcb/au-ar.sch (EAGLE design)
At the start: 74 parts, among them U1 TPD12S520DBTR, U2 TPD12S521DBTR

Commit message: added final edits for v1 order and pcbway gerbers
Parts:
- added FLASH: 0532610571, volks73-Molex:0532610571
- renumbered LINE_2_1 to 1, LINE_2_2 to 2, LINE_2_3 to 3, LINE_2_4 to 4
Connections:
- net 5V: no longer B1B.1, B1B.50, B1D.1, B1D.50
- net GND: now also FLASH-1.P$1
- net SPI_CLK: now also FLASH-2.P$1
- net SPI_CS: now also FLASH-5.P$1
- net SPI_DI: now also FLASH-3.P$1
- net SPI_DO: now also FLASH-4.P$1
Changed lines of the file:
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@@
 <part name="LINE_1_3" library="testpad" library_urn="urn:adsk.eagle:library:385" deviceset="TP" device="TP16R" package3d_urn="urn:adsk.eagle:package:27969/1"/>
 <part name="LINE_1_4" library="testpad" library_urn="urn:adsk.eagle:library:385" deviceset="TP" device="TP16R" package3d_urn="urn:adsk.eagle:package:27969/1"/>
-<part name="LINE_2_4" library="testpad" library_urn="urn:adsk.eagle:library:385" deviceset="TP" device="TP16R" package3d_urn="urn:adsk.eagle:package:27969/1" value="LINE_1"/>
-<part name="LINE_2_3" library="testpad" library_urn="urn:adsk.eagle:library:385" deviceset="TP" device="TP16R" package3d_urn="urn:adsk.eagle:package:27969/1" value="LINE_3"/>
-<part name="LINE_2_2" library="testpad" library_urn="urn:adsk.eagle:library:385" deviceset="TP" device="TP16R" package3d_urn="urn:adsk.eagle:package:27969/1" value="LINE_2"/>
-<part name="LINE_2_1" library="testpad" library_urn="urn:adsk.eagle:library:385" deviceset="TP" device="TP16R" package3d_urn="urn:adsk.eagle:package:27969/1" value="LINE_1"/>
+<part name="4" library="testpad" library_urn="urn:adsk.eagle:library:385" deviceset="TP" device="TP16R" package3d_urn="urn:adsk.eagle:package:27969/1" value="LINE_1"/>
+<part name="3" library="testpad" library_urn="urn:adsk.eagle:library:385" deviceset="TP" device="TP16R" package3d_urn="urn:adsk.eagle:package:27969/1" value="LINE_3"/>
+<part name="2" library="testpad" library_urn="urn:adsk.eagle:library:385" deviceset="TP" device="TP16R" package3d_urn="urn:adsk.eagle:package:27969/1" value="LINE_2"/>
+<part name="1" library="testpad" library_urn="urn:adsk.eagle:library:385" deviceset="TP" device="TP16R" package3d_urn="urn:adsk.eagle:package:27969/1" value="LINE_1"/>
 <part name="CAMERA1" library="S6B-PH-K-S_LF__SN_" deviceset="S6B-PH-K-S(LF)(SN)" device=""/>
 <part name="CAMERA2" library="S6B-PH-K-S_LF__SN_" deviceset="S6B-PH-K-S(LF)(SN)" device=""/>
@@
 <part name="R48" library="rcl" library_urn="urn:adsk.eagle:library:334" deviceset="R-US_" device="R0603" package3d_urn="urn:adsk.eagle:package:23555/3" value="47k"/>
 <part name="R49" library="rcl" library_urn="urn:adsk.eagle:library:334" deviceset="R-US_" device="R0603" package3d_urn="urn:adsk.eagle:package:23555/3" value="47k"/>
+<part name="FLASH" library="volks73-Molex" deviceset="0532610571" device=""/>
 </parts>
 <sheets>
@@
 </segment>
 <segment>
-<pinref part="B1" gate="B" pin="1"/>
-<wire x1="83.82" y1="91.44" x2="68.58" y2="91.44" width="0.1524" layer="91"/>
-<wire x1="68.58" y1="91.44" x2="68.58" y2="99.06" width="0.1524" layer="91"/>
-<label x="68.58" y="99.06" size="1.27" layer="95"/>
-</segment>
-<segment>
-<pinref part="B1" gate="B" pin="50"/>
-<wire x1="99.06" y1="91.44" x2="111.76" y2="91.44" width="0.1524" layer="91"/>
-<wire x1="111.76" y1="91.44" x2="111.76" y2="99.06" width="0.1524" layer="91"/>
-<label x="111.76" y="99.06" size="1.27" layer="95"/>
-</segment>
-<segment>
 <pinref part="B1" gate="C" pin="1"/>
 <wire x1="134.62" y1="91.44" x2="119.38" y2="91.44" width="0.1524" layer="91"/>
@@
 <wire x1="162.56" y1="91.44" x2="162.56" y2="99.06" width="0.1524" layer="91"/>
 <label x="162.56" y="99.06" size="1.27" layer="95"/>
-</segment>
-<segment>
-<pinref part="B1" gate="D" pin="1"/>
-<wire x1="187.96" y1="91.44" x2="172.72" y2="91.44" width="0.1524" layer="91"/>
-<wire x1="172.72" y1="91.44" x2="172.72" y2="99.06" width="0.1524" layer="91"/>
-<label x="172.72" y="99.06" size="1.27" layer="95"/>
-</segment>
-<segment>
-<pinref part="B1" gate="D" pin="50"/>
-<wire x1="203.2" y1="91.44" x2="215.9" y2="91.44" width="0.1524" layer="91"/>
-<wire x1="215.9" y1="91.44" x2="215.9" y2="99.06" width="0.1524" layer="91"/>
-<label x="215.9" y="99.06" size="1.27" layer="95"/>
 </segment>
 </net>
@@
 <attribute name="TP_SIGNAL_NAME" x="72.39" y="46.99" size="1.778" layer="97" rot="R180"/>
 </instance>
-<instance part="LINE_2_4" gate="G$1" x="170.18" y="45.72" smashed="yes" rot="R180">
+<instance part="4" gate="G$1" x="170.18" y="45.72" smashed="yes" rot="R180">
 <attribute name="TP_SIGNAL_NAME" x="168.91" y="46.99" size="1.778" layer="97" rot="R180"/>
 </instance>
-<instance part="LINE_2_3" gate="G$1" x="167.64" y="43.18" smashed="yes" rot="R180">
+<instance part="3" gate="G$1" x="167.64" y="43.18" smashed="yes" rot="R180">
 <attribute name="TP_SIGNAL_NAME" x="166.37" y="44.45" size="1.778" layer="97" rot="R180"/>
 </instance>
-<instance part="LINE_2_2" gate="G$1" x="170.18" y="40.64" smashed="yes" rot="R180">
+<instance part="2" gate="G$1" x="170.18" y="40.64" smashed="yes" rot="R180">
 <attribute name="TP_SIGNAL_NAME" x="168.91" y="41.91" size="1.778" layer="97" rot="R180"/>
 </instance>
-<instance part="LINE_2_1" gate="G$1" x="167.64" y="38.1" smashed="yes" rot="R180">
+<instance part="1" gate="G$1" x="167.64" y="38.1" smashed="yes" rot="R180">
 <attribute name="TP_SIGNAL_NAME" x="166.37" y="39.37" size="1.778" layer="97" rot="R180"/>
 </instance>
@@
 <segment>
 <pinref part="CAMERA2" gate="G$1" pin="1"/>
-<pinref part="LINE_2_4" gate="G$1" pin="TP"/>
+<pinref part="4" gate="G$1" pin="TP"/>
 <wire x1="172.72" y1="48.26" x2="170.18" y2="48.26" width="0.1524" layer="91"/>
 <pinref part="R7" gate="G$1" pin="2"/>
@@
 <segment>
 <pinref part="R8" gate="G$1" pin="2"/>
-<pinref part="LINE_2_3" gate="G$1" pin="TP"/>
+<pinref part="3" gate="G$1" pin="TP"/>
 <wire x1="152.4" y1="45.72" x2="167.64" y2="45.72" width="0.1524" layer="91"/>
 <pinref part="CAMERA2" gate="G$1" pin="2"/>
@@
 <segment>
 <pinref part="CAMERA2" gate="G$1" pin="3"/>
-<pinref part="LINE_2_2" gate="G$1" pin="TP"/>
+<pinref part="2" gate="G$1" pin="TP"/>
 <wire x1="172.72" y1="43.18" x2="170.18" y2="43.18" width="0.1524" layer="91"/>
 <pinref part="R9" gate="G$1" pin="2"/>
@@
 <segment>
 <pinref part="R10" gate="G$1" pin="2"/>
-<pinref part="LINE_2_1" gate="G$1" pin="TP"/>
+<pinref part="1" gate="G$1" pin="TP"/>
 <wire x1="162.56" y1="40.64" x2="167.64" y2="40.64" width="0.1524" layer="91"/>
 <pinref part="CAMERA2" gate="G$1" pin="4"/>
@@
 <attribute name="NAME" x="8.6614" y="36.83" size="1.778" layer="95" rot="R90"/>
 <attribute name="VALUE" x="13.462" y="36.83" size="1.778" layer="96" rot="R90"/>
+</instance>
+<instance part="FLASH" gate="-1" x="104.14" y="50.8" smashed="yes">
+<attribute name="NAME" x="104.14" y="53.34" size="1.778" layer="95"/>
+<attribute name="VALUE" x="104.14" y="45.72" size="1.778" layer="96"/>
+</instance>
+<instance part="FLASH" gate="-2" x="104.14" y="45.72" smashed="yes">
+<attribute name="NAME" x="104.14" y="48.26" size="1.778" layer="95"/>
+<attribute name="VALUE" x="104.14" y="40.64" size="1.778" layer="96"/>
+</instance>
+<instance part="FLASH" gate="-3" x="104.14" y="40.64" smashed="yes">
+<attribute name="NAME" x="104.14" y="43.18" size="1.778" layer="95"/>
+<attribute name="VALUE" x="104.14" y="35.56" size="1.778" layer="96"/>
+</instance>
+<instance part="FLASH" gate="-4" x="104.14" y="35.56" smashed="yes">
+<attribute name="NAME" x="104.14" y="38.1" size="1.778" layer="95"/>
+<attribute name="VALUE" x="104.14" y="30.48" size="1.778" layer="96"/>
+</instance>
+<instance part="FLASH" gate="-5" x="104.14" y="30.48" smashed="yes">
+<attribute name="NAME" x="104.14" y="33.02" size="1.778" layer="95"/>
+<attribute name="VALUE" x="104.14" y="25.4" size="1.778" layer="96"/>
 </instance>
 </instances>
@@
 <label x="15.24" y="5.08" size="1.27" layer="95"/>
 </segment>
+<segment>
+<wire x1="91.44" y1="45.72" x2="78.74" y2="45.72" width="0.1524" layer="91"/>
+<label x="68.58" y="45.72" size="1.778" layer="95"/>
+<pinref part="FLASH" gate="-1" pin="P$1"/>
+<wire x1="91.44" y1="45.72" x2="91.44" y2="50.8" width="0.1524" layer="91"/>
+<wire x1="91.44" y1="50.8" x2="99.06" y2="50.8" width="0.1524" layer="91"/>
+</segment>
 </net>
 <net name="SPI_CS" class="0">
@@
 <label x="0" y="33.02" size="1.27" layer="95"/>
 </segment>
+<segment>
+<wire x1="91.44" y1="35.56" x2="78.74" y2="35.56" width="0.1524" layer="91"/>
+<label x="68.58" y="35.56" size="1.778" layer="95"/>
+<pinref part="FLASH" gate="-5" pin="P$1"/>
+<wire x1="91.44" y1="35.56" x2="91.44" y2="30.48" width="0.1524" layer="91"/>
+<wire x1="91.44" y1="30.48" x2="99.06" y2="30.48" width="0.1524" layer="91"/>
+</segment>
 </net>
 <net name="SPI_DO" class="0">
@@
 <label x="0" y="27.94" size="1.27" layer="95"/>
 </segment>
+<segment>
+<wire x1="96.52" y1="38.1" x2="78.74" y2="38.1" width="0.1524" layer="91"/>
+<label x="68.58" y="38.1" size="1.778" layer="95"/>
+<wire x1="96.52" y1="38.1" x2="96.52" y2="35.56" width="0.1524" layer="91"/>
+<pinref part="FLASH" gate="-4" pin="P$1"/>
+<wire x1="96.52" y1="35.56" x2="99.06" y2="35.56" width="0.1524" layer="91"/>
+</segment>
 </net>
 <net name="SPI_CLK" class="0">
@@
 <label x="58.42" y="22.86" size="1.27" layer="95"/>
 </segment>
+<segment>
+<wire x1="96.52" y1="43.18" x2="78.74" y2="43.18" width="0.1524" layer="91"/>
+<label x="68.58" y="43.18" size="1.778" layer="95"/>
+<wire x1="96.52" y1="43.18" x2="96.52" y2="45.72" width="0.1524" layer="91"/>
+<pinref part="FLASH" gate="-2" pin="P$1"/>
+<wire x1="96.52" y1="45.72" x2="99.06" y2="45.72" width="0.1524" layer="91"/>
+</segment>
 </net>
 <net name="SPI_DI" class="0">
@@
 <label x="58.42" y="17.78" size="1.27" layer="95"/>
 </segment>
-</net>
+<segment>
+<wire x1="99.06" y1="40.64" x2="78.74" y2="40.64" width="0.1524" layer="91"/>
+<label x="68.58" y="40.64" size="1.778" layer="95"/>
+<pinref part="FLASH" gate="-3" pin="P$1"/>
+</segment>
+</net>

Commit message: added external oscillator
Parts:
- added C1: 0.1uF, rcl:C-USC0603
- added R27, R6: 3k, rcl:R-US_R0603
- added SI514: SI514, lupa300-components:SI514
Connections:
- new net OSC_CLK: B1C.45, SI514.CLK
- new net OSC_SCL: B1A.31, R27.1, SI514.SCL
- new net OSC_SDA: B1A.28, R6.1, SI514.SDA
- net 3V3: now also C1.1, R27.2, R6.2, SI514.VDD
- net CEC1_FPGA: now also B1C.37; no longer B1C.3
- net GND: now also C1.2, SI514.GND
Changed lines of the file:
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@@
 <?xml version="1.0" encoding="utf-8"?>
 <!DOCTYPE eagle SYSTEM "eagle.dtd">
-<eagle version="9.3.1">
+<eagle version="9.4.0">
 <drawing>
 <settings>
@@
 <part name="R49" library="rcl" library_urn="urn:adsk.eagle:library:334" deviceset="R-US_" device="R0603" package3d_urn="urn:adsk.eagle:package:23555/3" value="47k"/>
 <part name="FLASH" library="volks73-Molex" deviceset="0532610571" device=""/>
+<part name="SI514" library="lupa300-components" deviceset="SI514" device=""/>
+<part name="R6" library="rcl" library_urn="urn:adsk.eagle:library:334" deviceset="R-US_" device="R0603" package3d_urn="urn:adsk.eagle:package:23555/3" value="3k"/>
+<part name="R27" library="rcl" library_urn="urn:adsk.eagle:library:334" deviceset="R-US_" device="R0603" package3d_urn="urn:adsk.eagle:package:23555/3" value="3k"/>
+<part name="C1" library="rcl" library_urn="urn:adsk.eagle:library:334" deviceset="C-US" device="C0603" package3d_urn="urn:adsk.eagle:package:23616/2" value="0.1uF"/>
 </parts>
 <sheets>
@@
 <net name="CEC1_FPGA" class="0">
 <segment>
-<pinref part="B1" gate="C" pin="3"/>
-<wire x1="134.62" y1="86.36" x2="124.46" y2="86.36" width="0.1524" layer="91"/>
-<label x="116.84" y="86.36" size="1.27" layer="95"/>
+<pinref part="B1" gate="C" pin="37"/>
+<wire x1="149.86" y1="58.42" x2="160.02" y2="58.42" width="0.1524" layer="91"/>
+<label x="160.02" y="58.42" size="1.27" layer="95"/>
 </segment>
 </net>
@@
 <wire x1="48.26" y1="63.5" x2="58.42" y2="63.5" width="0.1524" layer="91"/>
 <label x="55.88" y="63.5" size="1.27" layer="95"/>
+</segment>
+</net>
+<net name="OSC_CLK" class="0">
+<segment>
+<pinref part="B1" gate="C" pin="45"/>
+<wire x1="149.86" y1="78.74" x2="160.02" y2="78.74" width="0.1524" layer="91"/>
+<label x="160.02" y="78.74" size="1.27" layer="95"/>
+</segment>
+</net>
+<net name="OSC_SDA" class="0">
+<segment>
+<pinref part="B1" gate="A" pin="28"/>
+<wire x1="48.26" y1="35.56" x2="58.42" y2="35.56" width="0.1524" layer="91"/>
+<label x="58.42" y="35.56" size="1.27" layer="95"/>
+</segment>
+</net>
+<net name="OSC_SCL" class="0">
+<segment>
+<pinref part="B1" gate="A" pin="31"/>
+<wire x1="48.26" y1="43.18" x2="58.42" y2="43.18" width="0.1524" layer="91"/>
+<label x="58.42" y="43.18" size="1.27" layer="95"/>
 </segment>
 </net>
@@
 </segment>
 </net>
+</nets>
+</sheet>
+<sheet>
+<description>Programmable Oscillator</description>
+<plain>
+</plain>
+<instances>
+<instance part="SI514" gate="G$1" x="22.86" y="20.32" smashed="yes">
+<attribute name="NAME" x="12.7" y="33.02" size="1.778" layer="95"/>
+<attribute name="VALUE" x="25.4" y="33.02" size="1.778" layer="96"/>
+</instance>
+<instance part="R6" gate="G$1" x="-10.16" y="30.48" smashed="yes" rot="R90">
+<attribute name="NAME" x="-11.6586" y="26.67" size="1.778" layer="95" rot="R90"/>
+<attribute name="VALUE" x="-6.858" y="26.67" size="1.778" layer="96" rot="R90"/>
+</instance>
+<instance part="R27" gate="G$1" x="-17.78" y="30.48" smashed="yes" rot="R90">
+<attribute name="NAME" x="-19.2786" y="26.67" size="1.778" layer="95" rot="R90"/>
+<attribute name="VALUE" x="-14.478" y="26.67" size="1.778" layer="96" rot="R90"/>
+</instance>
+<instance part="C1" gate="G$1" x="-27.94" y="30.48" smashed="yes">
+<attribute name="NAME" x="-26.924" y="31.115" size="1.778" layer="95"/>
+<attribute name="VALUE" x="-26.924" y="26.289" size="1.778" layer="96"/>
+</instance>
+</instances>
+<busses>
+</busses>
+<nets>
+<net name="3V3" class="0">
+<segment>
+<pinref part="SI514" gate="G$1" pin="VDD"/>
+<wire x1="10.16" y1="27.94" x2="2.54" y2="27.94" width="0.1524" layer="91"/>
+<label x="-5.08" y="27.94" size="1.778" layer="95"/>
+<pinref part="R6" gate="G$1" pin="2"/>
+<wire x1="2.54" y1="27.94" x2="2.54" y2="35.56" width="0.1524" layer="91"/>
+<wire x1="2.54" y1="35.56" x2="-10.16" y2="35.56" width="0.1524" layer="91"/>
+<pinref part="R27" gate="G$1" pin="2"/>
+<wire x1="-10.16" y1="35.56" x2="-17.78" y2="35.56" width="0.1524" layer="91"/>
+<junction x="-10.16" y="35.56"/>
+<pinref part="C1" gate="G$1" pin="1"/>
+<wire x1="-27.94" y1="33.02" x2="-27.94" y2="35.56" width="0.1524" layer="91"/>
+<wire x1="-27.94" y1="35.56" x2="-17.78" y2="35.56" width="0.1524" layer="91"/>
+<junction x="-17.78" y="35.56"/>
+</segment>
+</net>
+<net name="OSC_SDA" class="0">
+<segment>
+<pinref part="SI514" gate="G$1" pin="SDA"/>
+<label x="-5.08" y="22.86" size="1.778" layer="95"/>
+<wire x1="10.16" y1="22.86" x2="-10.16" y2="22.86" width="0.1524" layer="91"/>
+<pinref part="R6" gate="G$1" pin="1"/>
+<wire x1="-10.16" y1="22.86" x2="-10.16" y2="25.4" width="0.1524" layer="91"/>
+</segment>
+</net>
+<net name="OSC_SCL" class="0">
+<segment>
+<pinref part="SI514" gate="G$1" pin="SCL"/>
+<label x="-5.08" y="17.78" size="1.778" layer="95"/>
+<pinref part="R27" gate="G$1" pin="1"/>
+<wire x1="10.16" y1="17.78" x2="-17.78" y2="17.78" width="0.1524" layer="91"/>
+<wire x1="-17.78" y1="17.78" x2="-17.78" y2="25.4" width="0.1524" layer="91"/>
+</segment>
+</net>
+<net name="GND" class="0">
+<segment>
+<pinref part="SI514" gate="G$1" pin="GND"/>
+<label x="-5.08" y="12.7" size="1.778" layer="95"/>
+<pinref part="C1" gate="G$1" pin="2"/>
+<wire x1="-27.94" y1="25.4" x2="-27.94" y2="12.7" width="0.1524" layer="91"/>
+<wire x1="-27.94" y1="12.7" x2="10.16" y2="12.7" width="0.1524" layer="91"/>
+</segment>
+</net>
+<net name="OSC_CLK" class="0">
+<segment>
+<pinref part="SI514" gate="G$1" pin="CLK"/>
+<wire x1="35.56" y1="25.4" x2="40.64" y2="25.4" width="0.1524" layer="91"/>
+<label x="40.64" y="25.4" size="1.778" layer="95"/>
+</segment>
+</net>
