File: pcb/au-ar.sch (EAGLE design)
At the start: 57 parts, among them U1 TPD12S016PWR, U2 TPD12S016PWR

Commit message: added version from school pc
Parts:
- added U3: DMP3099L, gsynth:DMP3099L
- renumbered U$1 to U4
Connections:
- new net HP2_EN: B1A.40, U3.G
- net 5V: now also U3.D
- net HP2: now also U3.S
Changed lines of the file:
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@@
 <layer number="112" name="bGTest" color="7" fill="1" visible="yes" active="yes"/>
 <layer number="113" name="ReferenceLS" color="7" fill="1" visible="no" active="no"/>
+<layer number="114" name="Badge_Outline" color="7" fill="1" visible="yes" active="yes"/>
+<layer number="115" name="ReferenceISLANDS" color="7" fill="1" visible="yes" active="yes"/>
 <layer number="116" name="Patch_BOT" color="9" fill="4" visible="yes" active="yes"/>
 <layer number="118" name="Rect_Pads" color="7" fill="1" visible="no" active="no"/>
@@
 <part name="GND9" library="supply1" library_urn="urn:adsk.eagle:library:371" deviceset="GND" device=""/>
 <part name="GND10" library="supply1" library_urn="urn:adsk.eagle:library:371" deviceset="GND" device=""/>
-<part name="U$1" library="TDP12S521" deviceset="W25Q80DVSNIG" device=""/>
+<part name="U4" library="TDP12S521" deviceset="W25Q80DVSNIG" device=""/>
 <part name="R5" library="rcl" library_urn="urn:adsk.eagle:library:334" deviceset="R-US_" device="R0603" package3d_urn="urn:adsk.eagle:package:23555/3" value="47k"/>
 <part name="C11" library="rcl" library_urn="urn:adsk.eagle:library:334" deviceset="C-US" device="C0603" package3d_urn="urn:adsk.eagle:package:23616/2" value="0.1uF"/>
@@
 <part name="C4" library="rcl" library_urn="urn:adsk.eagle:library:334" deviceset="C-US" device="C0603" package3d_urn="urn:adsk.eagle:package:23616/2" value="0.1uF"/>
 <part name="C5" library="rcl" library_urn="urn:adsk.eagle:library:334" deviceset="C-US" device="C0603" package3d_urn="urn:adsk.eagle:package:23616/2" value="0.1uF"/>
+<part name="U3" library="gsynth" library_urn="urn:adsk.eagle:library:7741914" deviceset="DMP3099L" device="" package3d_urn="urn:adsk.eagle:package:7741968/1"/>
 </parts>
 <sheets>
@@
 </segment>
 </net>
+<net name="HP2_EN" class="0">
+<segment>
+<pinref part="B1" gate="A" pin="40"/>
+<wire x1="48.26" y1="66.04" x2="58.42" y2="66.04" width="0.1524" layer="91"/>
+<label x="58.42" y="66.04" size="1.778" layer="95"/>
+</segment>
+</net>
 </nets>
 </sheet>
@@
 <attribute name="VALUE" x="79.756" y="31.369" size="1.778" layer="96"/>
 </instance>
+<instance part="U3" gate="G$1" x="68.58" y="101.6" smashed="yes">
+<attribute name="NAME" x="73.66" y="101.6" size="1.778" layer="95" font="vector"/>
+<attribute name="VALUE" x="73.66" y="99.06" size="1.778" layer="96" font="vector"/>
+</instance>
 </instances>
 <busses>
@@
 </segment>
 </net>
-<net name="HP1" class="0">
-<segment>
-<pinref part="HDMI_1" gate="G$1" pin="19"/>
-<label x="12.7" y="45.72" size="1.778" layer="95"/>
-<wire x1="25.4" y1="45.72" x2="12.7" y2="45.72" width="0.1524" layer="91"/>
-</segment>
-</net>
 <net name="D22_P" class="1">
 <segment>
@@
 <pinref part="HDMI_2" gate="G$1" pin="19"/>
 <label x="81.28" y="43.18" size="1.778" layer="95"/>
-<wire x1="91.44" y1="43.18" x2="81.28" y2="43.18" width="0.1524" layer="91"/>
+<pinref part="U3" gate="G$1" pin="S"/>
+<wire x1="71.12" y1="96.52" x2="71.12" y2="43.18" width="0.1524" layer="91"/>
+<wire x1="71.12" y1="43.18" x2="91.44" y2="43.18" width="0.1524" layer="91"/>
 </segment>
 </net>
@@
 </segment>
 </net>
+<net name="5V" class="0">
+<segment>
+<pinref part="U3" gate="G$1" pin="D"/>
+<wire x1="71.12" y1="106.68" x2="71.12" y2="111.76" width="0.1524" layer="91"/>
+<label x="71.12" y="111.76" size="1.778" layer="95"/>
+</segment>
+</net>
+<net name="HP2_EN" class="0">
+<segment>
+<pinref part="U3" gate="G$1" pin="G"/>
+<wire x1="63.5" y1="99.06" x2="58.42" y2="99.06" width="0.1524" layer="91"/>
+<label x="55.88" y="99.06" size="1.778" layer="95"/>
+</segment>
+</net>
+<net name="HP1" class="0">
+<segment>
+<pinref part="HDMI_1" gate="G$1" pin="19"/>
+<wire x1="25.4" y1="45.72" x2="12.7" y2="45.72" width="0.1524" layer="91"/>
+<label x="12.7" y="45.72" size="1.778" layer="95"/>
+</segment>
+</net>
 </nets>
 </sheet>
@@
 </plain>
 <instances>
-<instance part="U$1" gate="G$1" x="25.4" y="15.24" smashed="yes">
+<instance part="U4" gate="G$1" x="25.4" y="15.24" smashed="yes">
 <attribute name="NAME" x="25.4" y="40.64" size="1.778" layer="95"/>
 <attribute name="VALUE" x="35.56" y="40.64" size="1.778" layer="96"/>
@@
 <net name="3V3" class="0">
 <segment>
-<pinref part="U$1" gate="G$1" pin="VCC"/>
+<pinref part="U4" gate="G$1" pin="VCC"/>
 <wire x1="50.8" y1="33.02" x2="58.42" y2="33.02" width="0.1524" layer="91"/>
 <wire x1="58.42" y1="33.02" x2="58.42" y2="48.26" width="0.1524" layer="91"/>
-<pinref part="U$1" gate="G$1" pin="HOLD"/>
+<pinref part="U4" gate="G$1" pin="HOLD"/>
 <wire x1="50.8" y1="27.94" x2="58.42" y2="27.94" width="0.1524" layer="91"/>
 <wire x1="58.42" y1="27.94" x2="58.42" y2="33.02" width="0.1524" layer="91"/>
 <junction x="58.42" y="33.02"/>
-<pinref part="U$1" gate="G$1" pin="WP"/>
+<pinref part="U4" gate="G$1" pin="WP"/>
 <wire x1="20.32" y1="22.86" x2="15.24" y2="22.86" width="0.1524" layer="91"/>
 <wire x1="15.24" y1="22.86" x2="15.24" y2="48.26" width="0.1524" layer="91"/>
@@
 <net name="GND" class="0">
 <segment>
-<pinref part="U$1" gate="G$1" pin="GND"/>
+<pinref part="U4" gate="G$1" pin="GND"/>
 <wire x1="20.32" y1="17.78" x2="15.24" y2="17.78" width="0.1524" layer="91"/>
 <wire x1="15.24" y1="17.78" x2="15.24" y2="5.08" width="0.1524" layer="91"/>
@@
 <net name="SPI_CS" class="0">
 <segment>
-<pinref part="U$1" gate="G$1" pin="CS"/>
+<pinref part="U4" gate="G$1" pin="CS"/>
 <wire x1="20.32" y1="33.02" x2="10.16" y2="33.02" width="0.1524" layer="91"/>
 <pinref part="R5" gate="G$1" pin="1"/>
@@
 <net name="SPI_DO" class="0">
 <segment>
-<pinref part="U$1" gate="G$1" pin="DO"/>
+<pinref part="U4" gate="G$1" pin="DO"/>
 <wire x1="20.32" y1="27.94" x2="7.62" y2="27.94" width="0.1524" layer="91"/>
 <label x="0" y="27.94" size="1.27" layer="95"/>
@@
 <net name="SPI_CLK" class="0">
 <segment>
-<pinref part="U$1" gate="G$1" pin="CLK"/>
+<pinref part="U4" gate="G$1" pin="CLK"/>
 <wire x1="50.8" y1="22.86" x2="58.42" y2="22.86" width="0.1524" layer="91"/>
 <label x="58.42" y="22.86" size="1.27" layer="95"/>
@@
 <net name="SPI_DI" class="0">
 <segment>
-<pinref part="U$1" gate="G$1" pin="DI"/>
+<pinref part="U4" gate="G$1" pin="DI"/>
 <wire x1="50.8" y1="17.78" x2="58.42" y2="17.78" width="0.1524" layer="91"/>
 <label x="58.42" y="17.78" size="1.27" layer="95"/>
