File: pcb/au-ar.brd (EAGLE design)
At the start: 65 x 45 mm, 59 parts, among them U1 TPD12S016PWR, U2 TPD12S016PWR

Commit message: v1.2 silk edits
Parts:
- moved C3 7.44 mm to (17.6, 40.0), turned to 90 degrees
- moved R13 0.26 mm to (46.7, 26.9)
- moved R14 0.17 mm to (46.6, 29.5)
- moved R12 0.15 mm to (46.6, 24.4)
- moved R28 0.10 mm to (15.0, 40.9)
- moved R4 0.08 mm to (51.6, 30.2)
Routing:
- net SCL2: track 21.0 -> 14.7 mm
- net 5V: track 24.9 -> 21.7 mm
- net LSOE2: track 19.0 -> 15.8 mm
- net OSC_SDA: track 38.2 -> 40.3 mm
- net CTHPD2: track 13.1 -> 11.9 mm
- net SDA2: track 21.1 -> 19.9 mm
- net GND: track 211.4 -> 212.2 mm
- net OSC_SCL: track 38.4 -> 39.1 mm
Other:
- board text added: "1"
- board text added: "2"
- board text added: "3"
- board text added: "4"
- board text added: "GND"
- board text added: "Matt Ruffner Dr. Daniel L. Lau Ying Yu University of Kentucky 2019"
- board text added: "Short SJ1 to enable HDMI output"
- board text removed: "Dr. Daniel L. Lau Matt Ruffner Ying Yu University of Kentucky 2019"

Commit message: final mods to v1.2 pcb and addition of v1.2 gerbers
Routing:
- net 3V3: track 112.3 -> 117.4 mm
- net GND: track 212.2 -> 215.5 mm
- net LINE_1_4: track 34.1 -> 34.8 mm
Changed lines of the file:
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@@
 <wire x1="41.461921875" y1="21.137190625" x2="41.461921875" y2="21.38045" width="0.2032" layer="1"/>
 <wire x1="41.461921875" y1="21.38045" x2="41.665121875" y2="21.58365" width="0.2032" layer="1"/>
-<wire x1="42.5323" y1="22.2123" x2="56.86586875" y2="36.54586875" width="0.2032" layer="1"/>
 <wire x1="56.86586875" y1="36.54586875" x2="56.8706" y2="36.54586875" width="0.2032" layer="1"/>
 <wire x1="36.322" y1="15.99726875" x2="36.322" y2="16.2433" width="0.2032" layer="1"/>
@@
 <wire x1="40.77335" y1="20.44861875" x2="40.77335" y2="20.69465" width="0.2032" layer="1"/>
 <wire x1="41.22893125" y1="20.9042" x2="41.461921875" y2="21.137190625" width="0.2032" layer="1"/>
-<wire x1="41.665121875" y1="21.58365" x2="41.90838125" y2="21.58365" width="0.2032" layer="1"/>
-<wire x1="41.90838125" y1="21.58365" x2="42.5323" y2="22.20756875" width="0.2032" layer="1"/>
-<wire x1="42.5323" y1="22.20756875" x2="42.5323" y2="22.2123" width="0.2032" layer="1"/>
+<wire x1="41.665121875" y1="21.58365" x2="41.90365" y2="21.58365" width="0.2032" layer="1"/>
+<wire x1="41.90365" y1="21.58365" x2="56.86586875" y2="36.54586875" width="0.2032" layer="1"/>
 </signal>
 <signal name="D11_P" class="1">
@@
 <wire x1="41.0277" y1="27.4828" x2="41.6373" y2="26.8732" width="0.2032" layer="16"/>
 <wire x1="43.6118" y1="26.8732" x2="44.83735" y2="25.64765" width="0.2032" layer="16"/>
-<wire x1="49.784" y1="26.7462" x2="49.784" y2="27.0002" width="0.2032" layer="16"/>
-<wire x1="48.68545" y1="25.64765" x2="49.784" y2="26.7462" width="0.2032" layer="16"/>
+<wire x1="53.2892" y1="26.6446" x2="53.51145" y2="26.42235" width="0.2032" layer="16"/>
+<wire x1="53.2892" y1="26.6446" x2="49.82845" y2="26.6446" width="0.2032" layer="16"/>
+<wire x1="48.8315" y1="25.64765" x2="49.82845" y2="26.6446" width="0.2032" layer="16"/>
 <wire x1="41.59285" y1="24.7142" x2="40.39905" y2="25.908" width="0.2032" layer="16"/>
 <wire x1="40.298" y1="25.908" x2="40.39905" y2="25.908" width="0.2032" layer="16"/>
 <wire x1="41.59285" y1="24.7142" x2="43.2067875" y2="24.7142" width="0.2032" layer="16"/>
 <wire x1="43.2067875" y1="24.7142" x2="44.8362875" y2="23.0847" width="0.2032" layer="16"/>
-<wire x1="49.5794125" y1="24.0538" x2="49.5794125" y2="24.4602" width="0.2032" layer="16"/>
-<wire x1="49.5794125" y1="24.0538" x2="48.6103125" y2="23.0847" width="0.2032" layer="16"/>
-<wire x1="44.8362875" y1="23.0847" x2="48.6103125" y2="23.0847" width="0.2032" layer="16"/>
+<wire x1="49.9667625" y1="22.6187" x2="48.1824125" y2="22.6187" width="0.2032" layer="16"/>
+<wire x1="48.1824125" y1="22.6187" x2="47.7164125" y2="23.0847" width="0.2032" layer="16"/>
+<wire x1="47.7164125" y1="23.0847" x2="44.8362875" y2="23.0847" width="0.2032" layer="16"/>
 <wire x1="40.298" y1="23.749" x2="43.9556" y2="20.0914" width="0.2032" layer="16"/>
 <wire x1="47.7012" y1="20.0914" x2="47.8282" y2="20.2184" width="0.2032" layer="16"/>
 <wire x1="47.7012" y1="20.0914" x2="43.9556" y2="20.0914" width="0.2032" layer="16"/>
 <via x="47.8282" y="20.2184" extent="1-16" drill="0.3"/>
-<via x="49.5794125" y="24.4602" extent="1-16" drill="0.3"/>
-<via x="49.784" y="27.0002" extent="1-16" drill="0.3"/>
+<via x="49.9667625" y="22.6187" extent="1-16" drill="0.3"/>
+<via x="53.51145" y="26.42235" extent="1-16" drill="0.3"/>
 <via x="56.3118" y="29.1846" extent="1-16" drill="0.3"/>
 <wire x1="40.298" y1="16.764" x2="41.441" y2="15.621" width="0.2032" layer="16"/>
@@
 <wire x1="17.64665" y1="41.91635" x2="17.60855" y2="41.95445" width="0.2032" layer="1"/>
 <via x="17.60855" y="41.95445" extent="1-16" drill="0.3"/>
-<wire x1="44.83735" y1="25.64765" x2="48.68545" y2="25.64765" width="0.2032" layer="16"/>
+<wire x1="44.83735" y1="25.64765" x2="48.8315" y2="25.64765" width="0.2032" layer="16"/>
 <wire x1="53.5" y1="42.7" x2="56.5" y2="42.7" width="0" layer="19" extent="16-16"/>
 <wire x1="56.5" y1="38.3" x2="53.5" y2="38.3" width="0" layer="19" extent="16-16"/>
@@
 <wire x1="46.8308375" y1="26.0604" x2="45.9608875" y2="26.93035" width="0.2032" layer="16"/>
 <wire x1="46.8308375" y1="26.0604" x2="48.3235" y2="26.0604" width="0.2032" layer="16"/>
-<wire x1="48.3235" y1="26.0604" x2="48.9331" y2="26.67" width="0.2032" layer="16"/>
-<wire x1="48.9331" y1="26.67" x2="48.9331" y2="26.76525" width="0.2032" layer="16"/>
-<via x="48.9331" y="26.76525" extent="1-16" drill="0.3"/>
-<via x="48.730871875" y="24.078284375" extent="1-16" drill="0.3"/>
-<wire x1="48.735584375" y1="24.073571875" x2="48.730871875" y2="24.078284375" width="0.2032" layer="16"/>
-<wire x1="48.1594625" y1="23.49745" x2="48.735584375" y2="24.073571875" width="0.2032" layer="16"/>
-<wire x1="46.58205" y1="23.49745" x2="48.1594625" y2="23.49745" width="0.2032" layer="16"/>
+<wire x1="48.3235" y1="26.0604" x2="49.32045" y2="27.05735" width="0.2032" layer="16"/>
+<wire x1="53.19395" y1="27.05735" x2="53.49875" y2="27.36215" width="0.2032" layer="16"/>
+<wire x1="53.19395" y1="27.05735" x2="49.32045" y2="27.05735" width="0.2032" layer="16"/>
+<via x="53.49875" y="27.36215" extent="1-16" drill="0.3"/>
+<via x="49.257921875" y="23.290884375" extent="1-16" drill="0.3"/>
+<wire x1="49.257921875" y1="23.290884375" x2="49.05135625" y2="23.49745" width="0.2032" layer="16"/>
+<wire x1="49.05135625" y1="23.49745" x2="46.58205" y2="23.49745" width="0.2032" layer="16"/>
 <wire x1="45.7082" y1="24.3713" x2="46.58205" y2="23.49745" width="0.2032" layer="16"/>
 <wire x1="45.7336" y1="21.7932" x2="45.7336" y2="20.71635" width="0.2032" layer="16"/>
@@
 <contactref element="R19" pad="2"/>
 <contactref element="B1" pad="AB_15"/>
-<wire x1="50.712" y1="23.622" x2="49.8212" y2="23.622" width="0.2032" layer="16"/>
-<wire x1="49.8212" y1="23.622" x2="47.9924" y2="21.7932" width="0.2032" layer="16"/>
-<wire x1="47.9924" y1="21.7932" x2="47.4336" y2="21.7932" width="0.2032" layer="16"/>
+<wire x1="50.712" y1="23.622" x2="50.712" y2="22.43635" width="0.2032" layer="16"/>
+<wire x1="50.712" y1="22.43635" x2="50.06885" y2="21.7932" width="0.2032" layer="16"/>
+<wire x1="50.06885" y1="21.7932" x2="47.4336" y2="21.7932" width="0.2032" layer="16"/>
 <wire x1="47.4336" y1="21.7932" x2="47.3955" y2="21.7932" width="0.2032" layer="16"/>
 <wire x1="47.3955" y1="21.7932" x2="46.5319" y2="22.6568" width="0.2032" layer="16"/>
@@
 <contactref element="LINE_1_3" pad="TP"/>
 <contactref element="CAMERA1" pad="2"/>
-<wire x1="58.166" y1="26.6926" x2="53.3236" y2="26.6926" width="0.2032" layer="16"/>
-<wire x1="53.3236" y1="26.6926" x2="52.412" y2="25.781" width="0.2032" layer="16"/>
+<wire x1="58.166" y1="26.6926" x2="57.49555" y2="26.6926" width="0.2032" layer="16"/>
+<wire x1="57.49555" y1="26.6926" x2="56.58395" y2="25.781" width="0.2032" layer="16"/>
+<wire x1="56.58395" y1="25.781" x2="52.412" y2="25.781" width="0.2032" layer="16"/>
 <wire x1="58.166" y1="26.6926" x2="57.2544" y2="25.781" width="0.2032" layer="1"/>
 <wire x1="57.2544" y1="25.781" x2="54.737" y2="25.781" width="0.2032" layer="1"/>
